Commit message: Fix collision for agv_mini_manipulator base in preparation for Gazebo.

File: agv_models/agv_mini_manipulator/agv_mini_manipulator_description/urdf/common_properties.xacro (robot description, xacro)
@@ -12,19 +12,5 @@
     </material>
     <!-- Common Xacros -->
-    <xacro:macro name="box" params="m o_xyz o_rpy link_name length width height">
-        <link name="${link_name}">
-            <visual>
-                <geometry>
-                <box size="${length} ${width} ${height}"/>
-                </geometry>
-                <origin xyz="${o_xyz}" rpy="${o_rpy}"/>
-                <material name="blue"/>
-            </visual>
-            <collision>
-                <geometry>
-                <box size="${length} ${width} ${height}"/>
-                </geometry>
-                <origin xyz="${o_xyz}" rpy="${o_rpy}"/>
-            </collision>
+    <xacro:macro name="box_inertia" params="m o_xyz o_rpy length width height">
             <inertial>
                 <mass value="${m}"/>
@@ -34,53 +20,22 @@
                          izz="${m /12 * (length**2 + width**2)}"/>
             </inertial>
-        </link>
     </xacro:macro>
-    <xacro:macro name="cylinder" params="link_name m radius length o_xyz o_rpy">
-        <link name="${link_name}">
-            <visual>
-                <geometry>
-                    <cylinder radius="${radius}" length="${length}"/>
-                </geometry>
-                <origin xyz="${o_xyz}" rpy="${o_rpy}"/>
-                <material name="black"/>
-            </visual>
-            <collision>
-                <geometry>
-                    <cylinder radius="${radius}" length="${length}"/>
-                </geometry>
-                <origin xyz="${o_xyz}" rpy="${o_rpy}"/>
-            </collision>
-            <inertial>
-                <mass value="${m}"/>
-                <origin xyz="${o_xyz}" rpy="${o_rpy}"/>
-                <inertia ixx="${m / 12 * (3*radius**2 + length**2)}" ixy="0" ixz="0"
-                         iyy="${m / 12 * (3*radius**2 + length**2)}" iyz="0"
-                         izz="${m / 2 * radius**2}"/>
-            </inertial>
-        </link>
+    <xacro:macro name="cylinder_inertia" params="m radius length o_xyz o_rpy">
+        <inertial>
+            <mass value="${m}"/>
+            <origin xyz="${o_xyz}" rpy="${o_rpy}"/>
+            <inertia ixx="${m / 12 * (3*radius**2 + length**2)}" ixy="0" ixz="0"
+                        iyy="${m / 12 * (3*radius**2 + length**2)}" iyz="0"
+                        izz="${m / 2 * radius**2}"/>
+        </inertial>
     </xacro:macro>
-    <xacro:macro name="sphere" params="link_name m radius o_xyz o_rpy">
-        <link name="${link_name}">
-            <visual>
-                <geometry>
-                <sphere radius="${radius}"/>
-                </geometry>
-                <origin xyz="${o_xyz}" rpy="${o_rpy}"/>
-                <material name="gray"/>
-            </visual>
-            <collision>
-                <geometry>
-                <sphere radius="${radius}"/>
-                </geometry>
-                <origin xyz="${o_xyz}" rpy="${o_rpy}"/>
-            </collision>
-            <inertial>
-                <mass value="${m}"/>
-                <origin xyz="${o_xyz}" rpy="${o_rpy}"/>
-                <inertia ixx="${2/3 * m * (radius)**2}" ixy="0" ixz="0"
-                         iyy="${2/3 * m * (radius)**2}" iyz="0"
-                         izz="${2/3 * m * (radius)**2}"/>
-            </inertial>
-        </link>
+    <xacro:macro name="sphere_inertia" params="m radius o_xyz o_rpy">
+        <inertial>
+            <mass value="${m}"/>
+            <origin xyz="${o_xyz}" rpy="${o_rpy}"/>
+            <inertia ixx="${2/5 * m * (radius)**2}" ixy="0" ixz="0"
+                     iyy="${2/5 * m * (radius)**2}" iyz="0"
+                     izz="${2/5 * m * (radius)**2}"/>
+        </inertial>
     </xacro:macro>
     <!-- Joint Xacros -->

File: agv_models/agv_mini_manipulator/agv_mini_manipulator_description/urdf/mobile_base/mobile_base.xacro (robot description, xacro)
@@ -14,5 +14,5 @@
     <!-- base_footprint_base_link_joint -->
     <link name="base_footprint"/>
-    <xacro:box m="5.0" o_xyz="0 0 0" o_rpy="0 0 0"
+    <xacro:robot_base m="5.0" o_xyz="0 0 0" o_rpy="0 0 0"
     link_name="base_link" length="${base_length}"
     width="${base_width}" height="${base_height}"/>

File: agv_models/agv_mini_manipulator/agv_mini_manipulator_description/urdf/mobile_base/mobile_base_macros.xacro (robot description, xacro)
@@ -1,18 +1,82 @@
 <?xml version ="1.0"?>
 <robot xmlns:xacro="http://www.ros.org/wiki/xacro">
+    <xacro:macro name="robot_base" params="link_name m o_xyz o_rpy length width height">
+        <link name="${link_name}">
+            <visual>
+                <geometry>
+                <box size="${length} ${width} ${height}"/>
+                </geometry>
+                <origin xyz="${o_xyz}" rpy="${o_rpy}"/>
+                <material name="blue"/>
+            </visual>
+            <collision>
+                <geometry>
+                <box size="${length} ${width} ${height}"/>
+                </geometry>
+                <origin xyz="${o_xyz}" rpy="${o_rpy}"/>
+            </collision>
+            <xacro:box_inertia m="${m}" o_xyz="${o_xyz}" o_rpy="${o_rpy}"
+            length="${length}" width="${width}" height="${height}"/>
+        </link>
+    </xacro:macro>
     <xacro:macro name="lidar" params="prefix m lidar_radius lidar_height">
-        <xacro:cylinder link_name="${prefix}_lidar_link" m="${m}"
-                        radius="${lidar_radius}" length="${lidar_height}"
-                        o_xyz="0 0 0" o_rpy="0 0 0"/>
+        <link name="${prefix}_lidar_link">
+            <visual>
+                <geometry>
+                    <cylinder radius="${lidar_radius}" length="${lidar_height}"/>
+                </geometry>
+                <origin xyz="0 0 0" rpy="0 0 0"/>
+                <material name="black"/>
+            </visual>
+            <collision>
+                <geometry>
+                    <cylinder radius="${lidar_radius}" length="${lidar_height}"/>
+                </geometry>
+                <origin xyz="0 0 0" rpy="0 0 0"/>
+            </collision>
+            <xacro:cylinder_inertia
+            m="${m}" radius="${lidar_radius}" length="${lidar_height}"
+            o_xyz="0 0 0" o_rpy="0 0 0"/>
+        </link>
     </xacro:macro>
     <xacro:macro name="wheel" params="m prefix wheel_radius wheel_thickness">
-        <xacro:cylinder link_name="${prefix}_wheel_link" m="${m}"
-                        radius="${wheel_radius}" length="${wheel_thickness}"
-                        o_xyz="0 0 0" o_rpy="0 0 0"/>
+        <link name="${prefix}_wheel_link">
+            <visual>
+                <geometry>
+                    <cylinder radius="${wheel_radius}" length="${wheel_thickness}"/>
+                </geometry>
+                <origin xyz="0 0 0" rpy="0 0 0"/>
+                <material name="black"/>
+            </visual>
+            <collision>
+                <geometry>
+                <sphere radius="${wheel_radius}"/>
+                </geometry>
+                <origin xyz="0 0 0" rpy="0 0 0"/>
+            </collision>
+            <xacro:cylinder_inertia
+            m="${m}" radius="${wheel_radius}" length="${wheel_thickness }"
+            o_xyz="0 0 0" o_rpy="0 0 0"/>
+        </link>
     </xacro:macro>
     <xacro:macro name="castor_wheel" params="prefix m wheel_offset">
-        <xacro:sphere link_name="${prefix}_castor_wheel_link" m="${m}"
-                        radius="${wheel_offset/2.0}"
-                        o_xyz="0 0 0" o_rpy="0 0 0"/>
+        <link name="${prefix}_castor_wheel_link">
+            <visual>
+                <geometry>
+                <sphere radius="${wheel_offset/2.0}"/>
+                </geometry>
+                <origin xyz="0 0 0" rpy="0 0 0"/>
+                <material name="gray"/>
+            </visual>
+            <collision>
+                <geometry>
+                <sphere radius="${wheel_offset/2.0}"/>
+                </geometry>
+                <origin xyz="0 0 0" rpy="0 0 0"/>
+            </collision>
+            <xacro:sphere_inertia
+            m="${m}" radius="${wheel_offset/2.0}"
+            o_xyz="0 0 0" o_rpy="0 0 0"/>
+        </link>
     </xacro:macro>
 </robot>
