Commit message: Break apart agv_mini_manipulator xacro to component and foundational xacros. Correct inertias.

File: agv_models/agv_mini_manipulator/agv_mini_manipulator_description/urdf/agv_mini_manipulator.urdf.xacro (robot description, xacro)
@@ -1,199 +1,6 @@
 <?xml version ="1.0"?>
 <robot name="agv_mini_manipulator" xmlns:xacro="http://www.ros.org/wiki/xacro">
-    <!-- Variables -->
-    <xacro:property name="base_length" value="0.5"/>
-    <xacro:property name="base_width" value="0.4"/>
-    <xacro:property name="base_height" value="0.2"/>
-    <xacro:property name="wheel_offset" value="0.075"/>
-    <xacro:property name="wheel_thickness" value="0.05"/>
-    <xacro:property name="wheel_radius" value="0.1"/>
-    <xacro:property name="lidar_height" value="0.03"/>
-    <xacro:property name="lidar_radius" value="0.03"/>
-    <!-- Materials -->
-    <material name="blue">
-        <color rgba="0 0 1 1"/>
-    </material>
-    <material name="black">
-        <color rgba="0 0 0 1"/>
-    </material>
-    <material name="gray">
-        <color rgba="0.5 0.5 0.5 1"/>
-    </material>
-    <!-- Macro definitions -->
-    <xacro:macro name="lidar" params="prefix">
-        <link name="${prefix}_lidar_link">
-            <visual>
-                <geometry>
-                    <cylinder radius="${lidar_radius}" length="${lidar_height}"/>
-                </geometry>
-                <origin xyz="0 0 ${lidar_height / 2.0}" rpy="0 0 0"/>
-                <material name="black"/>
-            </visual>
-            <collision>
-                <geometry>
-                    <cylinder radius="${lidar_radius}" length="${lidar_height}"/>
-                </geometry>
-                <origin xyz="0 0 ${lidar_height / 2.0}" rpy="0 0 0"/>
-            </collision>
-            <inertial>
-                <mass value="5.0"/>
-                <origin xyz="0 0 0" rpy="0 0 0"/>
-                <inertia ixx="0.1" ixy="0" ixz="0" iyy="0.1" iyz="0" izz="0.1"/>
-            </inertial>
-        </link>
-    </xacro:macro>
-    <xacro:macro name="wheel" params="prefix">
-        <link name="${prefix}_wheel_link">
-            <visual>
-                <geometry>
-                    <cylinder radius="${wheel_radius}"
-                    length="${wheel_thickness}"/>
-                </geometry>
-                <origin xyz="0 0 0" rpy="0 0 0"/>
-                <material name="gray"/>
-            </visual>
-            <collision>
-                <geometry>
-                    <cylinder radius="${wheel_radius}"
-                    length="${wheel_thickness}"/>
-                </geometry>
-                <origin xyz="0 0 0" rpy="0 0 0"/>
-            </collision>
-            <inertial>
-                <mass value="5.0"/>
-                <origin xyz="0 0 0" rpy="0 0 0"/>
-                <inertia ixx="0.1" ixy="0" ixz="0" iyy="0.1" iyz="0" izz="0.1"/>
-            </inertial>
-        </link>
-    </xacro:macro>
-    <xacro:macro name="castor_wheel" params="prefix">
-        <link name="${prefix}_castor_wheel_link">
-            <visual>
-                <geometry>
-                <sphere radius="${wheel_offset/2.0}"/>
-                </geometry>
-                <origin xyz="0 0 0" rpy="0 0 0"/>
-                <material name="gray"/>
-            </visual>
-            <collision>
-                <geometry>
-                <sphere radius="${wheel_offset/2.0}"/>
-                </geometry>
-                <origin xyz="0 0 0" rpy="0 0 0"/>
-            </collision>
-            <inertial>
-                <mass value="5.0"/>
-                <origin xyz="0 0 0" rpy="0 0 0"/>
-                <inertia ixx="0.1" ixy="0" ixz="0" iyy="0.1" iyz="0" izz="0.1"/>
-            </inertial>
-        </link>
-    </xacro:macro>
-    <xacro:macro name="three_axis_joint" params="prefix parent_link">
-        <link name="${prefix}_link_x"/>
-        <joint name="${prefix}_joint_x" type="continuous">
-            <parent link="${parent_link}"/>
-            <child link="${prefix}_link_x"/>
-            <origin xyz="0 0 0" rpy="0 0 0"/>
-            <axis xyz="1 0 0"/>
-        </joint>
-        <link name="${prefix}_link_y"/>
-        <joint name="${prefix}_joint_y" type="continuous">
-            <parent link="${prefix}_link_x"/>
-            <child link="${prefix}_link_y"/>
-            <origin xyz="0 0 0" rpy="0 0 0"/>
-            <axis xyz="0 1 0"/>
-        </joint>
-        <link name="${prefix}_link_z"/>
-        <joint name="${prefix}_joint_z" type="continuous">
-            <parent link="${prefix}_link_y"/>
-            <child link="${prefix}_link_z"/>
-            <origin xyz="0 0 0" rpy="0 0 0"/>
-            <axis xyz="0 0 1"/>
-        </joint>
-    </xacro:macro>
-    <!-- base_footprint_base_link_joint -->
-    <link name="base_footprint"/>
-    <link name="base_link">
-    <visual>
-        <geometry>
-        <box size="${base_length} ${base_width} ${base_height}"/>
-        </geometry>
-        <origin xyz="0 0 0" rpy="0 0 0"/>
-        <material name="blue"/>
-    </visual>
-    <collision>
-        <geometry>
-        <box size="${base_length} ${base_width} ${base_height}"/>
-        </geometry>
-        <origin xyz="0 0 0" rpy="0 0 0"/>
-    </collision>
-    <inertial>
-        <mass value="5.0"/>
-        <origin xyz="0 0 0" rpy="0 0 0"/>
-        <inertia ixx="0.1" ixy="0" ixz="0" iyy="0.1" iyz="0" izz="0.1"/>
-    </inertial>
-    </link>
-    <joint name="base_footprint_base_link_joint" type="fixed">
-        <parent link="base_footprint"/>
-        <child link="base_link"/>
-        <origin xyz="0 0 ${base_height / 2.0 + wheel_offset}" rpy="0 0 0"/>
-    </joint>
-    <!-- base_footprint_base_link_joint -->
-    <!-- base_link_lidar_front_joint -->
-    <xacro:lidar prefix="front"/>
-    <joint name="base_link_lidar_front_joint" type="fixed">
-        <parent link="base_link"/>
-        <child link="front_lidar_link"/>
-        <origin xyz="${base_length / 2.0 - 0.05} 0.0 ${base_height / 2.0}" rpy="0 0 0"/>
-    </joint>
-    <!-- base_link_lidar_front_joint -->
-    <!-- base_link_lidar_back_joint -->
-    <xacro:lidar prefix="back"/>
-    <joint name="base_link_lidar_back_joint" type="fixed">
-        <parent link="base_link"/>
-        <child link="back_lidar_link"/>
-        <origin xyz="${-1.0*(base_length / 2.0 - 0.05)} 0.0 ${base_height / 2.0}"
-        rpy="0 0 ${pi / 2.0}"/>
-    </joint>
-    <!-- base_link_lidar_back_joint -->
-    <!-- base_link_right_wheel_joint -->
-    <xacro:wheel prefix="right"/>
-    <joint name="base_link_right_wheel_joint" type="continuous">
-        <parent link="base_link"/>
-        <child link="right_wheel_link"/>
-        <origin xyz="0.0 ${base_width / 2.0 + wheel_thickness / 2.0} ${-1.0 * (base_height / 2.0 - wheel_radius + wheel_offset)}"
-        rpy="${-pi / 2.0} 0 0"/>
-        <axis xyz="0 1 0"/>
-    </joint>
-    <!-- base_link_right_wheel_joint -->
-    <!-- base_link_left_wheel_joint -->
-    <xacro:wheel prefix="left"/>
-    <joint name="base_link_left_wheel_joint" type="continuous">
-        <parent link="base_link"/>
-        <child link="left_wheel_link"/>
-        <origin xyz="0.0 ${-1.0*(base_width / 2.0 + wheel_thickness / 2.0)} ${-1.0 * (base_height / 2.0 - wheel_radius + wheel_offset)}"
-        rpy="${pi / 2.0} 0 0"/>
-        <axis xyz="0 1 0"/>
-    </joint>
-    <!-- base_link_left_wheel_joint -->
-    <!-- base_link_front_wheel_joint -->
-    <xacro:castor_wheel prefix="front"/>
-    <joint name="base_link_front_wheel_joint" type="fixed">
-        <parent link="base_link"/>
-        <child link="front_castor_wheel_link"/>
-        <origin xyz="${base_length / 2.0 - 0.075} 0.0 ${-1.0*(base_height / 2.0 + wheel_offset / 2.0)}"
-        rpy="0 0 0"/>
-    </joint>
-    <xacro:three_axis_joint prefix="front_castor_wheel" parent_link="front_castor_wheel_link"/>
-    <!-- base_link_front_wheel_joint -->
-    <!-- base_link_back_wheel_joint -->
-    <xacro:castor_wheel prefix="back"/>
-    <joint name="base_link_back_wheel_joint" type="fixed">
-        <parent link="base_link"/>
-        <child link="back_castor_wheel_link"/>
-        <origin xyz="${-1.0*(base_length / 2.0 - 0.075)} 0.0 ${-1.0*(base_height / 2.0 + wheel_offset / 2.0)}"
-        rpy="0 0 0"/>
-    </joint>
-    <xacro:three_axis_joint prefix="back_castor_wheel" parent_link="back_castor_wheel_link"/>
-    <!-- base_link_back_wheel_joint -->
+    <xacro:include filename="common_properties.xacro"/>
+    <!-- Mobile Base-->
+    <xacro:include filename="$(find agv_mini_manipulator_description)/urdf/mobile_base/mobile_base.xacro"/>
 </robot>

Commit message: Add Gazebo launch file and bridge to agv_mini_manipulator_bringup. Add Gazebo xacro to agv_mini_manipulator_description.

File: agv_models/agv_mini_manipulator/agv_mini_manipulator_description/urdf/agv_mini_manipulator.urdf.xacro (robot description, xacro)
@@ -4,3 +4,5 @@
     <!-- Mobile Base-->
     <xacro:include filename="$(find agv_mini_manipulator_description)/urdf/mobile_base/mobile_base.xacro"/>
+    <!-- Gazebo -->
+    <xacro:include filename="$(find agv_mini_manipulator_description)/urdf/mobile_base/mobile_base_gazebo.xacro"/>
 </robot>

File: agv_models/agv_mini_manipulator/agv_mini_manipulator_description/urdf/common_properties.xacro (robot description, xacro)
@@ -40,6 +40,17 @@
     </xacro:macro>
     <!-- Joint Xacros -->
+    <xacro:macro name="nonzero_inertia">
+        <inertial>
+            <mass value="0.0001"/>
+            <origin xyz="0 0 0" rpy="0 0 0"/>
+            <inertia ixx="1e-6" ixy="0" ixz="0"
+                     iyy="1e-6" iyz="0"
+                     izz="1e-6"/>
+        </inertial>
+    </xacro:macro>
     <xacro:macro name="three_axis_joint" params="prefix parent_link">
-        <link name="${prefix}_link_x"/>
+        <link name="${prefix}_link_x">
+            <xacro:nonzero_inertia/>
+        </link>
         <joint name="${prefix}_joint_x" type="continuous">
             <parent link="${parent_link}"/>
@@ -48,5 +59,7 @@
             <axis xyz="1 0 0"/>
         </joint>
-        <link name="${prefix}_link_y"/>
+        <link name="${prefix}_link_y">
+            <xacro:nonzero_inertia/>
+        </link>
         <joint name="${prefix}_joint_y" type="continuous">
             <parent link="${prefix}_link_x"/>
@@ -55,5 +68,7 @@
             <axis xyz="0 1 0"/>
         </joint>
-        <link name="${prefix}_link_z"/>
+        <link name="${prefix}_link_z">
+            <xacro:nonzero_inertia/>
+        </link>
         <joint name="${prefix}_joint_z" type="continuous">
             <parent link="${prefix}_link_y"/>

File: agv_models/agv_mini_manipulator/agv_mini_manipulator_description/urdf/mobile_base/mobile_base.xacro (robot description, xacro)
@@ -47,6 +47,6 @@
         <child link="right_wheel_link"/>
         <origin xyz="0.0 ${base_width / 2.0 + wheel_thickness / 2.0} ${-1.0 * (base_height / 2.0 - wheel_radius + wheel_offset)}"
-        rpy="${-pi / 2.0} 0 0"/>
-        <axis xyz="0 1 0"/>
+        rpy="${pi / 2.0} 0 0"/>
+        <axis xyz="0 0 1"/>
     </joint>
     <!-- base_link_right_wheel_joint -->
@@ -58,9 +58,9 @@
         <origin xyz="0.0 ${-1.0*(base_width / 2.0 + wheel_thickness / 2.0)} ${-1.0 * (base_height / 2.0 - wheel_radius + wheel_offset)}"
         rpy="${pi / 2.0} 0 0"/>
-        <axis xyz="0 1 0"/>
+        <axis xyz="0 0 1"/>
     </joint>
     <!-- base_link_left_wheel_joint -->
     <!-- base_link_front_wheel_joint -->
-    <xacro:castor_wheel m="0.75" prefix="front" wheel_offset="${wheel_offset}"/>
+    <xacro:castor_wheel prefix="front" m="0.75" wheel_offset="${wheel_offset}"/>
     <joint name="base_link_front_wheel_joint" type="fixed">
         <parent link="base_link"/>
@@ -72,5 +72,5 @@
     <!-- base_link_front_wheel_joint -->
     <!-- base_link_back_wheel_joint -->
-    <xacro:castor_wheel m="0.75" prefix="back" wheel_offset="${wheel_offset}"/>
+    <xacro:castor_wheel prefix="back" m="0.75" wheel_offset="${wheel_offset}"/>
     <joint name="base_link_back_wheel_joint" type="fixed">
         <parent link="base_link"/>

Commit message: Add world to agv_mini_manipulator bringup. Add camera to agv_mini_manipulator and make sensors separate xacro files.

File: agv_models/agv_mini_manipulator/agv_mini_manipulator_description/urdf/agv_mini_manipulator.urdf.xacro (robot description, xacro)
@@ -4,4 +4,7 @@
     <!-- Mobile Base-->
     <xacro:include filename="$(find agv_mini_manipulator_description)/urdf/mobile_base/mobile_base.xacro"/>
+    <!-- Sensors -->
+    <xacro:include filename="$(find agv_mini_manipulator_description)/urdf/sensors/camera.xacro"/>
+    <xacro:include filename="$(find agv_mini_manipulator_description)/urdf/sensors/lidar.xacro"/>
     <!-- Gazebo -->
     <xacro:include filename="$(find agv_mini_manipulator_description)/urdf/mobile_base/mobile_base_gazebo.xacro"/>

File: agv_models/agv_mini_manipulator/agv_mini_manipulator_description/urdf/common_properties.xacro (robot description, xacro)
@@ -44,7 +44,7 @@
             <mass value="0.0001"/>
             <origin xyz="0 0 0" rpy="0 0 0"/>
-            <inertia ixx="1e-6" ixy="0" ixz="0"
-                     iyy="1e-6" iyz="0"
-                     izz="1e-6"/>
+            <inertia ixx="1e-9" ixy="0" ixz="0"
+                     iyy="1e-9" iyz="0"
+                     izz="1e-9"/>
         </inertial>
     </xacro:macro>

File: agv_models/agv_mini_manipulator/agv_mini_manipulator_description/urdf/mobile_base/mobile_base.xacro (robot description, xacro)
@@ -10,11 +10,10 @@
     <xacro:property name="wheel_thickness" value="0.05"/>
     <xacro:property name="wheel_radius" value="0.1"/>
-    <xacro:property name="lidar_height" value="0.03"/>
-    <xacro:property name="lidar_radius" value="0.03"/>
     <!-- base_footprint_base_link_joint -->
     <link name="base_footprint"/>
-    <xacro:robot_base m="5.0" o_xyz="0 0 0" o_rpy="0 0 0"
+    <xacro:box_link m="5.0" o_xyz="0 0 0" o_rpy="0 0 0"
     link_name="base_link" length="${base_length}"
-    width="${base_width}" height="${base_height}"/>
+    width="${base_width}" height="${base_height}"
+    material_name="blue"/>
     <joint name="base_footprint_base_link_joint" type="fixed">
         <parent link="base_footprint"/>
@@ -23,22 +22,4 @@
     </joint>
     <!-- base_footprint_base_link_joint -->
-    <!-- base_link_lidar_front_joint -->
-    <xacro:lidar prefix="front" m="0.5" lidar_radius="${lidar_radius}" lidar_height="${lidar_height}"/>
-    <joint name="base_link_lidar_front_joint" type="fixed">
-        <parent link="base_link"/>
-        <child link="front_lidar_link"/>
-        <origin xyz="${base_length / 2.0 - 0.05} 0.0 ${base_height / 2.0 + lidar_height / 2.0}"
-        rpy="0 0 0"/>
-    </joint>
-    <!-- base_link_lidar_front_joint -->
-    <!-- base_link_lidar_back_joint -->
-    <xacro:lidar prefix="back" m="0.5" lidar_radius="${lidar_radius}" lidar_height="${lidar_height}"/>
-    <joint name="base_link_lidar_back_joint" type="fixed">
-        <parent link="base_link"/>
-        <child link="back_lidar_link"/>
-        <origin xyz="${-1.0*(base_length / 2.0 - 0.05)} 0.0 ${base_height / 2.0 + lidar_height / 2.0}"
-        rpy="0 0 ${pi / 2.0}"/>
-    </joint>
-    <!-- base_link_lidar_back_joint -->
     <!-- base_link_right_wheel_joint -->
     <xacro:wheel prefix="right" m="2.0" wheel_radius="${wheel_radius}" wheel_thickness="${wheel_thickness}"/>

File: agv_models/agv_mini_manipulator/agv_mini_manipulator_description/urdf/mobile_base/mobile_base_macros.xacro (robot description, xacro)
@@ -1,5 +1,5 @@
 <?xml version ="1.0"?>
 <robot xmlns:xacro="http://www.ros.org/wiki/xacro">
-    <xacro:macro name="robot_base" params="link_name m o_xyz o_rpy length width height">
+    <xacro:macro name="box_link" params="link_name m o_xyz o_rpy length width height material_name">
         <link name="${link_name}">
             <visual>
@@ -8,5 +8,5 @@
                 </geometry>
                 <origin xyz="${o_xyz}" rpy="${o_rpy}"/>
-                <material name="blue"/>
+                <material name="${material_name}"/>
             </visual>
             <collision>
