Commit message: agv_mini_manipulator xacro refactor. Add agv_mini_manipulator manipulator xacro.

File: agv_models/agv_mini_manipulator/agv_mini_manipulator_description/urdf/agv_mini_manipulator.urdf.xacro (robot description, xacro)
@@ -2,10 +2,12 @@
 <robot name="agv_mini_manipulator" xmlns:xacro="http://www.ros.org/wiki/xacro">
     <xacro:include filename="common_properties.xacro"/>
+    <xacro:include filename="common_hardware.xacro"/>
     <!-- Mobile Base-->
-    <xacro:include filename="$(find agv_mini_manipulator_description)/urdf/mobile_base/mobile_base.xacro"/>
+    <!-- <xacro:include filename="$(find agv_mini_manipulator_description)/urdf/mobile_base/mobile_base.xacro"/> -->
+    <!-- <xacro:include filename="$(find agv_mini_manipulator_description)/urdf/mobile_base/mobile_base_gazebo.xacro"/> -->
     <!-- Sensors -->
-    <xacro:include filename="$(find agv_mini_manipulator_description)/urdf/sensors/camera.xacro"/>
-    <xacro:include filename="$(find agv_mini_manipulator_description)/urdf/sensors/lidar.xacro"/>
-    <!-- Gazebo -->
-    <xacro:include filename="$(find agv_mini_manipulator_description)/urdf/mobile_base/mobile_base_gazebo.xacro"/>
+    <!-- <xacro:include filename="$(find agv_mini_manipulator_description)/urdf/sensors/camera.xacro"/> -->
+    <!-- <xacro:include filename="$(find agv_mini_manipulator_description)/urdf/sensors/lidar.xacro"/> -->
+    <!-- Manipulator -->
+    <xacro:include filename="$(find agv_mini_manipulator_description)/urdf/manipulator/manipulator.xacro"/>
 </robot>

File: agv_models/agv_mini_manipulator/agv_mini_manipulator_description/urdf/common_properties.xacro (robot description, xacro)
@@ -11,4 +11,7 @@
         <color rgba="0.5 0.5 0.5 1"/>
     </material>
+    <material name="orange">
+        <color rgba="1 0.5 0 1"/>
+    </material>
     <!-- Common Xacros -->
     <xacro:macro name="box_inertia" params="m o_xyz o_rpy length width height">
@@ -21,4 +24,23 @@
             </inertial>
     </xacro:macro>
+    <xacro:macro name="box_link" params="link_name m o_xyz o_rpy length width height material_name">
+        <link name="${link_name}">
+            <visual>
+                <geometry>
+                <box size="${length} ${width} ${height}"/>
+                </geometry>
+                <origin xyz="${o_xyz}" rpy="${o_rpy}"/>
+                <material name="${material_name}"/>
+            </visual>
+            <collision>
+                <geometry>
+                <box size="${length} ${width} ${height}"/>
+                </geometry>
+                <origin xyz="${o_xyz}" rpy="${o_rpy}"/>
+            </collision>
+            <xacro:box_inertia m="${m}" o_xyz="${o_xyz}" o_rpy="${o_rpy}"
+            length="${length}" width="${width}" height="${height}"/>
+        </link>
+    </xacro:macro>
     <xacro:macro name="cylinder_inertia" params="m radius length o_xyz o_rpy">
         <inertial>
@@ -30,4 +52,24 @@
         </inertial>
     </xacro:macro>
+    <xacro:macro name="cylinder" params="link_name m o_xyz o_rpy radius length material_name">
+        <link name="${link_name}">
+            <visual>
+                <geometry>
+                    <cylinder radius="${radius}" length="${length}"/>
+                </geometry>
+                <origin xyz="${o_xyz}" rpy="${o_rpy}"/>
+                <material name="${material_name}"/>
+            </visual>
+            <collision>
+                <geometry>
+                    <cylinder radius="${radius}" length="${length}"/>
+                </geometry>
+                <origin xyz="${o_xyz}" rpy="${o_rpy}"/>
+            </collision>
+            <xacro:cylinder_inertia
+            m="${m}" radius="${radius}" length="${length}"
+            o_xyz="${o_xyz}" o_rpy="${o_rpy}"/>
+        </link>
+    </xacro:macro>
     <xacro:macro name="sphere_inertia" params="m radius o_xyz o_rpy">
         <inertial>
@@ -38,4 +80,24 @@
                      izz="${2/5 * m * (radius)**2}"/>
         </inertial>
+    </xacro:macro>
+    <xacro:macro name="sphere" params="link_name m o_xyz o_rpy radius material_name">
+        <link name="${link_name}">
+            <visual>
+                <geometry>
+                <sphere radius="${radius}"/>
+                </geometry>
+                <origin xyz="${o_xyz}" rpy="${o_rpy}"/>
+                <material name="${material_name}"/>
+            </visual>
+            <collision>
+                <geometry>
+                <sphere radius="${radius}"/>
+                </geometry>
+                <origin xyz="${o_xyz}" rpy="${o_rpy}"/>
+            </collision>
+            <xacro:sphere_inertia
+            m="${m}" radius="${radius}"
+            o_xyz="${o_xyz}" o_rpy="${o_rpy}"/>
+        </link>
     </xacro:macro>
     <!-- Joint Xacros -->

File: agv_models/agv_mini_manipulator/agv_mini_manipulator_description/urdf/mobile_base/mobile_base.xacro (robot description, xacro)
@@ -1,6 +1,4 @@
 <?xml version ="1.0"?>
 <robot xmlns:xacro="http://www.ros.org/wiki/xacro">
-    <!-- Macros -->
-    <xacro:include filename="mobile_base_macros.xacro"/>
     <!-- Variables -->
     <xacro:property name="base_length" value="0.5"/>
@@ -12,7 +10,6 @@
     <!-- base_footprint_base_link_joint -->
     <link name="base_footprint"/>
-    <xacro:box_link m="5.0" o_xyz="0 0 0" o_rpy="0 0 0"
-    link_name="base_link" length="${base_length}"
-    width="${base_width}" height="${base_height}"
+    <xacro:box_link link_name="base_link" m="5.0" o_xyz="0 0 0" o_rpy="0 0 0"
+    length="${base_length}" width="${base_width}" height="${base_height}"
     material_name="blue"/>
     <joint name="base_footprint_base_link_joint" type="fixed">
@@ -23,5 +20,5 @@
     <!-- base_footprint_base_link_joint -->
     <!-- base_link_right_wheel_joint -->
-    <xacro:wheel prefix="right" m="2.0" wheel_radius="${wheel_radius}" wheel_thickness="${wheel_thickness}"/>
+    <xacro:wheel prefix="right" m="2.0" o_xyz="0 0 0" o_rpy="0 0 0" wheel_radius="${wheel_radius}" wheel_thickness="${wheel_thickness}"/>
     <joint name="base_link_right_wheel_joint" type="continuous">
         <parent link="base_link"/>
@@ -33,5 +30,5 @@
     <!-- base_link_right_wheel_joint -->
     <!-- base_link_left_wheel_joint -->
-    <xacro:wheel prefix="left" m="2.0" wheel_radius="${wheel_radius}" wheel_thickness="${wheel_thickness}"/>
+    <xacro:wheel prefix="left" m="2.0" o_xyz="0 0 0" o_rpy="0 0 0" wheel_radius="${wheel_radius}" wheel_thickness="${wheel_thickness}"/>
     <joint name="base_link_left_wheel_joint" type="continuous">
         <parent link="base_link"/>
@@ -43,5 +40,6 @@
     <!-- base_link_left_wheel_joint -->
     <!-- base_link_front_wheel_joint -->
-    <xacro:castor_wheel prefix="front" m="0.75" wheel_offset="${wheel_offset}"/>
+    <xacro:sphere link_name="front_castor_wheel_link" m="0.75" o_xyz="0 0 0" o_rpy="0 0 0"
+    radius="${wheel_offset/2.0}" material_name="black"/>
     <joint name="base_link_front_wheel_joint" type="fixed">
         <parent link="base_link"/>
@@ -53,5 +51,6 @@
     <!-- base_link_front_wheel_joint -->
     <!-- base_link_back_wheel_joint -->
-    <xacro:castor_wheel prefix="back" m="0.75" wheel_offset="${wheel_offset}"/>
+    <xacro:sphere link_name="back_castor_wheel_link" m="0.75" o_xyz="0 0 0" o_rpy="0 0 0"
+    radius="${wheel_offset/2.0}" material_name="black"/>
     <joint name="base_link_back_wheel_joint" type="fixed">
         <parent link="base_link"/>

File: agv_models/agv_mini_manipulator/agv_mini_manipulator_description/urdf/mobile_base/mobile_base_gazebo.xacro (robot description, xacro)
@@ -1,8 +1,4 @@
 <?xml version ="1.0"?>
 <robot xmlns:xacro="http://www.ros.org/wiki/xacro">
-    <!-- Variables -->
-    <xacro:property name="base_width" value="0.5"/>
-    <xacro:property name="wheel_thickness" value="0.05"/>
-    <xacro:property name="wheel_radius" value="0.1"/>
     <gazebo reference="front_castor_wheel_link">
         <mu1>0.1</mu1>

File: agv_models/agv_mini_manipulator/agv_mini_manipulator_description/urdf/sensors/lidar.xacro (robot description, xacro)
@@ -5,5 +5,6 @@
     <xacro:property name="lidar_radius" value="0.03"/>
     <!-- base_link_lidar_front_joint -->
-    <xacro:lidar prefix="front" m="0.5" lidar_radius="${lidar_radius}" lidar_height="${lidar_height}"/>
+    <xacro:cylinder link_name="front_lidar_link" m="0.5" o_xyz="0 0 0" o_rpy="0 0 0"
+    radius="${lidar_radius}" length="${lidar_height}" material_name="black"/>
     <joint name="base_link_lidar_front_joint" type="fixed">
         <parent link="base_link"/>
@@ -14,5 +15,6 @@
     <!-- base_link_lidar_front_joint -->
     <!-- base_link_lidar_back_joint -->
-    <xacro:lidar prefix="back" m="0.5" lidar_radius="${lidar_radius}" lidar_height="${lidar_height}"/>
+    <xacro:cylinder link_name="back_lidar_link" m="0.5" o_xyz="0 0 0" o_rpy="0 0 0"
+    radius="${lidar_radius}" length="${lidar_height}" material_name="black"/>
     <joint name="base_link_lidar_back_joint" type="fixed">
         <parent link="base_link"/>
