Commit message: Add rgb camera to agv_mini_manipulator.

File: agv_models/agv_mini_manipulator/agv_mini_manipulator_description/urdf/sensors/camera.xacro (robot description, xacro)
@@ -6,11 +6,44 @@
    <!-- base_link_rgbd_camera_joint -->
     <xacro:box_link m="0.5" o_xyz="0 0 0" o_rpy="0 0 0"
-    link_name="rgbd_camera_link" length="${camera_length}"
+    link_name="rgb_camera_link" length="${camera_length}"
     width="${camera_width}" height="${camera_height}" material_name="gray"/>
     <joint name="base_link_rgbd_camera_joint" type="fixed">
         <parent link="base_link"/>
-        <child link="rgbd_camera_link"/>
+        <child link="rgb_camera_link"/>
         <origin xyz="${base_length / 2.0 + camera_length / 2.0} 0 0" rpy="0 0 0"/>
     </joint>
     <!-- base_link_rgbd_camera_joint -->
+    <link name="rgb_camera_optical_link"/>
+    <joint name="rgb_camera_optical_joint" type="fixed">
+        <parent link="rgb_camera_link"/>
+        <child link="rgb_camera_optical_link"/>
+        <origin xyz="0 0 0" rpy="${-pi/2.0} 0 ${-pi/2.0}"/>
+    </joint>
+    <gazebo reference="rgb_camera_link">
+        <sensor type="camera" name="rgbd_camera">
+            <camera>
+                <horizontal_fov>1.3962634</horizontal_fov>
+                <image>
+                    <width>640</width>
+                    <height>480</height>
+                    <format>R8G8B8</format>
+                </image>
+                <clip>
+                    <near>0.1</near>
+                    <far>15</far>
+                </clip>
+                <noise>
+                    <type>gaussian</type>
+                    <mean>0.0</mean>
+                    <stddev>0.007</stddev>
+                </noise>
+                <optical_frame_id>rgb_camera_optical_link</optical_frame_id>
+                <camera_info_topic>camera/camera_info</camera_info_topic>
+            </camera>
+            <always_on>1</always_on>
+            <update_rate>20</update_rate>
+            <visualize>true</visualize>
+            <topic>camera/image_raw</topic>
+        </sensor>
+    </gazebo>
 </robot>
