Commit message: agv_mini_manipulator lidar angles.

File: agv_models/agv_mini_manipulator/agv_mini_manipulator_description/urdf/sensors/lidar.xacro (robot description, xacro)
@@ -13,8 +13,7 @@
         rpy="0 0 0"/>
     </joint>
-    <!-- base_link_lidar_front_joint -->
     <gazebo reference="front_lidar_link">
         <sensor name="front_lidar_link" type="gpu_lidar">
-                <topic>laser_scan</topic>
+                <topic>scan_front</topic>
                 <visualize>true</visualize>
                 <update_rate>10</update_rate>
@@ -23,19 +22,63 @@
                     <scan>
                         <horizontal>
-                        <samples>10</samples>
-                        <resolution>1</resolution>
-                        <min_angle>${-pi / 2.0}</min_angle>
-                        <max_angle>${pi / 2.0}</max_angle>
+                            <samples>20</samples>
+                            <resolution>1</resolution>
+                            <min_angle>${-5*pi / 8.0}</min_angle>
+                            <max_angle>${5*pi / 8.0}</max_angle>
                         </horizontal>
-                        <vertical>
-                        <samples>4</samples>
-                        <resolution>1</resolution>
-                        <min_angle>-0.261799</min_angle>
-                        <max_angle>0.261799</max_angle>
-                        </vertical>
+                        <!-- <vertical>
+                            <samples>4</samples>
+                            <resolution>1</resolution>
+                            <min_angle>-0.261799</min_angle>
+                            <max_angle>0.261799</max_angle>
+                        </vertical> -->
                     </scan>
                     <range>
                         <min>0.05</min>
-                        <max>100</max>
+                        <max>15</max>
+                        <resolution>0.01</resolution>
+                    </range>
+                    <noise>
+                        <type>gaussian</type>
+                        <mean>0</mean>
+                        <stddev>0.01</stddev>
+                    </noise>
+                </lidar>
+            </sensor>
+    </gazebo>
+    <!-- base_link_lidar_front_joint -->
+    <!-- base_link_lidar_back_joint -->
+    <xacro:cylinder link_name="back_lidar_link" m="0.5" o_xyz="0 0 0" o_rpy="0 0 0"
+    radius="${lidar_radius}" length="${lidar_height}" material_name="black"/>
+    <joint name="base_link_lidar_back_joint" type="fixed">
+        <parent link="base_link"/>
+        <child link="back_lidar_link"/>
+        <origin xyz="${-1.0*(base_length / 2.0 - 0.05)} 0.0 ${base_height / 2.0 + lidar_height / 2.0}"
+        rpy="0 0 ${pi / 2.0}"/>
+    </joint>
+    <gazebo reference="back_lidar_link">
+        <sensor name="back_lidar_link" type="gpu_lidar">
+                <topic>scan_back</topic>
+                <visualize>true</visualize>
+                <update_rate>10</update_rate>
+                <gz_frame_id>back_lidar_link</gz_frame_id>
+                <lidar>
+                    <scan>
+                        <horizontal>
+                            <samples>20</samples>
+                            <resolution>1</resolution>
+                            <min_angle>${-1*pi / 8.0}</min_angle>
+                            <max_angle>${9*pi / 8.0}</max_angle>
+                        </horizontal>
+                        <!-- <vertical>
+                            <samples>4</samples>
+                            <resolution>1</resolution>
+                            <min_angle>-0.261799</min_angle>
+                            <max_angle>0.261799</max_angle>
+                        </vertical> -->
+                    </scan>
+                    <range>
+                        <min>0.05</min>
+                        <max>15</max>
                         <resolution>0.01</resolution>
                     </range>
@@ -49,12 +92,3 @@
     </gazebo>
     <!-- base_link_lidar_back_joint -->
-    <xacro:cylinder link_name="back_lidar_link" m="0.5" o_xyz="0 0 0" o_rpy="0 0 0"
-    radius="${lidar_radius}" length="${lidar_height}" material_name="black"/>
-    <joint name="base_link_lidar_back_joint" type="fixed">
-        <parent link="base_link"/>
-        <child link="back_lidar_link"/>
-        <origin xyz="${-1.0*(base_length / 2.0 - 0.05)} 0.0 ${base_height / 2.0 + lidar_height / 2.0}"
-        rpy="0 0 ${pi / 2.0}"/>
-    </joint>
-    <!-- base_link_lidar_back_joint -->
 </robot>
