Commit message: agv_mini_manipulator file structure renaming. Separated arm and mobile base urdfs and launch.

File: agv_models/agv_mini_manipulator/agv_mini_manipulator_description/urdf/manipulator/arm.xacro (robot description, xacro)
@@ -10,4 +10,6 @@
     <xacro:property name="q1_limit_effort" value="100"/>
     <xacro:property name="q1_limit_velocity" value="100.0"/>
+    <xacro:property name="q1_friction" value="0.3"/>
+    <xacro:property name="q1_damping" value="0.3"/>
     <xacro:property name="q2_length" value="0.132"/>
     <xacro:property name="q2_limit_lower" value="${-3*pi / 4.0}"/>
@@ -15,4 +17,6 @@
     <xacro:property name="q2_limit_effort" value="100"/>
     <xacro:property name="q2_limit_velocity" value="100.0"/>
+    <xacro:property name="q2_friction" value="0.3"/>
+    <xacro:property name="q2_damping" value="0.3"/>
     <xacro:property name="q3_length" value="0.132"/>
     <xacro:property name="q3_limit_lower" value="${-3*pi / 4.0}"/>
@@ -20,13 +24,15 @@
     <xacro:property name="q3_limit_effort" value="100"/>
     <xacro:property name="q3_limit_velocity" value="100.0"/>
-    <!-- manipulator_base_link -->
-    <xacro:cylinder link_name="manipulator_base_link" m="2.0" o_xyz="0 0 ${q1_height / 2.0}"
+    <xacro:property name="q3_friction" value="0.3"/>
+    <xacro:property name="q3_damping" value="0.3"/>
+    <!-- arm_base_link -->
+    <xacro:cylinder link_name="arm_base_link" m="2.0" o_xyz="0 0 ${q1_height / 2.0}"
     o_rpy="0 0 0" radius="0.06" length="${q1_height}" material_name="orange"/>
-    <!-- manipulator_base_link -->
+    <!-- arm_base_link -->
     <!-- q1 -->
     <xacro:sphere link_name="q1_link" m="0.75" o_xyz="0 0 0" o_rpy="0 0 0"
     radius="0.05" material_name="orange"/>
     <joint name="q1" type="revolute">
-        <parent link="manipulator_base_link"/>
+        <parent link="arm_base_link"/>
         <child link="q1_link"/>
         <origin xyz="0 0 ${q1_height + manipulator_link_width / 2.0}" rpy="0 0 0"/>
@@ -34,4 +40,5 @@
         <limit lower="${q1_limit_lower}" upper="${q1_limit_upper}"
         effort="${q1_limit_effort}" velocity="${q1_limit_velocity}"/>
+        <dynamics damping="${q1_damping}" friction="${q1_friction}"/>
     </joint>
     <!-- q1 -->
@@ -47,4 +54,5 @@
         <limit lower="${q2_limit_lower}" upper="${q2_limit_upper}"
         effort="${q2_limit_effort}" velocity="${q2_limit_velocity}"/>
+        <dynamics damping="${q2_damping}" friction="${q2_friction}"/>
     </joint>
     <!-- q2 -->
@@ -61,4 +69,5 @@
         <limit lower="${q3_limit_lower}" upper="${q3_limit_upper}"
         effort="${q3_limit_effort}" velocity="${q3_limit_velocity}"/>
+        <dynamics damping="${q3_damping}" friction="${q3_friction}"/>
     </joint>
     <!-- q3 -->

Commit message: Add ros-gazebo bridge for agv_mini_manipulator arm. Change arm home position.

File: agv_models/agv_mini_manipulator/agv_mini_manipulator_description/urdf/manipulator/arm.xacro (robot description, xacro)
@@ -5,7 +5,14 @@
     <xacro:property name="manipulator_link_thickness" value="0.02"/>
     <xacro:property name="manipulator_joint_offset" value="0.01"/>
-    <xacro:property name="q1_height" value="0.05"/>
-    <xacro:property name="q1_limit_lower" value="${-3*pi / 4.0}"/>
-    <xacro:property name="q1_limit_upper" value="${3*pi / 4.0}"/>
+    <xacro:property name="q0_height" value="0.05"/>
+    <xacro:property name="q0_limit_lower" value="${-3*pi / 4.0}"/>
+    <xacro:property name="q0_limit_upper" value="${3*pi / 4.0}"/>
+    <xacro:property name="q0_limit_effort" value="100"/>
+    <xacro:property name="q0_limit_velocity" value="100.0"/>
+    <xacro:property name="q0_friction" value="0.3"/>
+    <xacro:property name="q0_damping" value="0.3"/>
+    <xacro:property name="q1_length" value="0.132"/>
+    <xacro:property name="q1_limit_lower" value="${-pi / 4.0}"/>
+    <xacro:property name="q1_limit_upper" value="${pi / 2.0}"/>
     <xacro:property name="q1_limit_effort" value="100"/>
     <xacro:property name="q1_limit_velocity" value="100.0"/>
@@ -14,27 +21,34 @@
     <xacro:property name="q2_length" value="0.132"/>
     <xacro:property name="q2_limit_lower" value="${-3*pi / 4.0}"/>
-    <xacro:property name="q2_limit_upper" value="0.0"/>
+    <xacro:property name="q2_limit_upper" value="${3*pi / 4.0}"/>
     <xacro:property name="q2_limit_effort" value="100"/>
     <xacro:property name="q2_limit_velocity" value="100.0"/>
     <xacro:property name="q2_friction" value="0.3"/>
     <xacro:property name="q2_damping" value="0.3"/>
-    <xacro:property name="q3_length" value="0.132"/>
-    <xacro:property name="q3_limit_lower" value="${-3*pi / 4.0}"/>
-    <xacro:property name="q3_limit_upper" value="${3*pi / 4.0}"/>
-    <xacro:property name="q3_limit_effort" value="100"/>
-    <xacro:property name="q3_limit_velocity" value="100.0"/>
-    <xacro:property name="q3_friction" value="0.3"/>
-    <xacro:property name="q3_damping" value="0.3"/>
     <!-- arm_base_link -->
-    <xacro:cylinder link_name="arm_base_link" m="2.0" o_xyz="0 0 ${q1_height / 2.0}"
-    o_rpy="0 0 0" radius="0.06" length="${q1_height}" material_name="orange"/>
+    <xacro:cylinder link_name="arm_base_link" m="2.0" o_xyz="0 0 ${q0_height / 2.0}"
+    o_rpy="0 0 0" radius="0.06" length="${q0_height}" material_name="orange"/>
     <!-- arm_base_link -->
+    <!-- q0 -->
+    <xacro:sphere link_name="q0_link" m="0.75" o_xyz="0 0 0" o_rpy="0 0 0"
+    radius="0.05" material_name="orange"/>
+    <joint name="q0" type="revolute">
+        <parent link="arm_base_link"/>
+        <child link="q0_link"/>
+        <origin xyz="0 0 ${q0_height + manipulator_link_width / 2.0}" rpy="0 0 0"/>
+        <axis xyz="0 0 1"/>
+        <limit lower="${q0_limit_lower}" upper="${q0_limit_upper}"
+        effort="${q0_limit_effort}" velocity="${q0_limit_velocity}"/>
+        <dynamics damping="${q0_damping}" friction="${q0_friction}"/>
+    </joint>
+    <!-- q0 -->
     <!-- q1 -->
-    <xacro:sphere link_name="q1_link" m="0.75" o_xyz="0 0 0" o_rpy="0 0 0"
-    radius="0.05" material_name="orange"/>
+    <xacro:box_link link_name="q1_link" m="0.5" o_xyz="${q1_length / 2.0} 0 0"
+    o_rpy="0 0 0" length="${q1_length + manipulator_joint_offset}" width="${manipulator_link_width}"
+    height="${manipulator_link_thickness}" material_name="orange"/>
     <joint name="q1" type="revolute">
-        <parent link="arm_base_link"/>
+        <parent link="q0_link"/>
         <child link="q1_link"/>
-        <origin xyz="0 0 ${q1_height + manipulator_link_width / 2.0}" rpy="0 0 0"/>
+        <origin xyz="0 0 0" rpy="${-pi / 2.0} ${-pi / 2.0} 0"/>
         <axis xyz="0 0 1"/>
         <limit lower="${q1_limit_lower}" upper="${q1_limit_upper}"
@@ -50,5 +64,6 @@
         <parent link="q1_link"/>
         <child link="q2_link"/>
-        <origin xyz="0 0 0" rpy="${-pi / 2.0} 0 0"/>
+        <origin xyz="${q2_length - manipulator_joint_offset} 0 ${manipulator_link_thickness}"
+        rpy="0 0 0"/>
         <axis xyz="0 0 1"/>
         <limit lower="${q2_limit_lower}" upper="${q2_limit_upper}"
@@ -57,18 +72,3 @@
     </joint>
     <!-- q2 -->
-    <!-- q3 -->
-    <xacro:box_link link_name="q3_link" m="0.5" o_xyz="${q3_length / 2.0} 0 0"
-    o_rpy="0 0 0" length="${q3_length + manipulator_joint_offset}" width="${manipulator_link_width}"
-    height="${manipulator_link_thickness}" material_name="orange"/>
-    <joint name="q3" type="revolute">
-        <parent link="q2_link"/>
-        <child link="q3_link"/>
-        <origin xyz="${q2_length - manipulator_joint_offset} 0 ${manipulator_link_thickness}"
-        rpy="0 0 0"/>
-        <axis xyz="0 0 1"/>
-        <limit lower="${q3_limit_lower}" upper="${q3_limit_upper}"
-        effort="${q3_limit_effort}" velocity="${q3_limit_velocity}"/>
-        <dynamics damping="${q3_damping}" friction="${q3_friction}"/>
-    </joint>
-    <!-- q3 -->
 </robot>

File: agv_models/agv_mini_manipulator/agv_mini_manipulator_description/urdf/manipulator/arm_gazebo.xacro (robot description, xacro)
@@ -2,4 +2,11 @@
 <robot xmlns:xacro="http://www.ros.org/wiki/xacro">
     <!-- Controllers -->
+    <gazebo>
+        <plugin
+            filename="gz-sim-joint-position-controller-system"
+            name="gz::sim::systems::JointPositionController" >
+            <joint_name>q0</joint_name>
+        </plugin>
+    </gazebo>
     <gazebo>
         <plugin
@@ -16,11 +23,4 @@
         </plugin>
     </gazebo>
-    <gazebo>
-        <plugin
-            filename="gz-sim-joint-position-controller-system"
-            name="gz::sim::systems::JointPositionController" >
-            <joint_name>q3</joint_name>
-        </plugin>
-    </gazebo>
     <!-- State publisher -->
     <gazebo>
@@ -28,7 +28,7 @@
             filename="gz-sim-joint-state-publisher-system"
             name="gz::sim::systems::JointStatePublisher" >
+            <joint_name>q0</joint_name>
             <joint_name>q1</joint_name>
             <joint_name>q2</joint_name>
-            <joint_name>q3</joint_name>
         </plugin>
     </gazebo>

File: agv_models/agv_mini_manipulator/agv_mini_manipulator_description/urdf/robot.urdf.xacro (robot description, xacro)
@@ -6,4 +6,4 @@
     <!-- <xacro:include filename="$(find agv_mini_manipulator_description)/urdf/mobile_base/mobile_base_robot.urdf.xacro"/> -->
     <!-- Manipulator -->
-    <xacro:include filename="$(find agv_mini_manipulator_description)/urdf/manipulator/manipulator.urdf.xacro"/>
+    <!-- <xacro:include filename="$(find agv_mini_manipulator_description)/urdf/manipulator/manipulator.urdf.xacro"/> -->
 </robot>

Commit message: Fix agv_mini_manipulator mobile base gazebo-ros bridge.

File: agv_models/agv_mini_manipulator/agv_mini_manipulator_description/urdf/manipulator/arm.xacro (robot description, xacro)
@@ -4,5 +4,5 @@
     <xacro:property name="manipulator_link_width" value="0.04"/>
     <xacro:property name="manipulator_link_thickness" value="0.02"/>
-    <xacro:property name="manipulator_joint_offset" value="0.01"/>
+    <xacro:property name="manipulator_joint_offset" value="0.02"/>
     <xacro:property name="q0_height" value="0.05"/>
     <xacro:property name="q0_limit_lower" value="${-3*pi / 4.0}"/>
@@ -27,5 +27,5 @@
     <xacro:property name="q2_damping" value="0.3"/>
     <!-- arm_base_link -->
-    <xacro:cylinder link_name="arm_base_link" m="2.0" o_xyz="0 0 ${q0_height / 2.0}"
+    <xacro:cylinder link_name="arm_base_link" m="10.0" o_xyz="0 0 ${q0_height / 2.0}"
     o_rpy="0 0 0" radius="0.06" length="${q0_height}" material_name="orange"/>
     <!-- arm_base_link -->

File: agv_models/agv_mini_manipulator/agv_mini_manipulator_description/urdf/manipulator/arm_gazebo.xacro (robot description, xacro)
@@ -7,4 +7,5 @@
             name="gz::sim::systems::JointPositionController" >
             <joint_name>q0</joint_name>
+            <p_gain>5.0</p_gain>
         </plugin>
     </gazebo>
@@ -14,4 +15,5 @@
             name="gz::sim::systems::JointPositionController" >
             <joint_name>q1</joint_name>
+            <p_gain>3.0</p_gain>
         </plugin>
     </gazebo>
@@ -21,4 +23,5 @@
             name="gz::sim::systems::JointPositionController" >
             <joint_name>q2</joint_name>
+            <p_gain>3.0</p_gain>
         </plugin>
     </gazebo>

File: agv_models/agv_mini_manipulator/agv_mini_manipulator_description/urdf/mobile_base/mobile_base_robot.urdf.xacro (robot description, xacro)
@@ -1,4 +1,6 @@
 <?xml version ="1.0"?>
 <robot name="agv_mini_manipulator_mobile_base" xmlns:xacro="http://www.ros.org/wiki/xacro">
+    <xacro:include filename="$(find agv_mini_manipulator_description)/urdf/common_properties.xacro"/>
+    <xacro:include filename="$(find agv_mini_manipulator_description)/urdf/common_hardware.xacro"/>
     <!-- Mobile Base-->
     <xacro:include filename="$(find agv_mini_manipulator_description)/urdf/mobile_base/mobile_base.xacro"/>

Commit message: Merge agv_mini_manipulator arm and mobile base together.

File: agv_models/agv_mini_manipulator/agv_mini_manipulator_description/urdf/manipulator/arm.xacro (robot description, xacro)
@@ -2,7 +2,7 @@
 <robot xmlns:xacro="http://www.ros.org/wiki/xacro">
     <!-- Variables -->
-    <xacro:property name="manipulator_link_width" value="0.04"/>
-    <xacro:property name="manipulator_link_thickness" value="0.02"/>
-    <xacro:property name="manipulator_joint_offset" value="0.02"/>
+    <xacro:property name="manipulator_link_width" value="0.08"/>
+    <xacro:property name="manipulator_link_thickness" value="0.04"/>
+    <xacro:property name="manipulator_joint_offset" value="0.04"/>
     <xacro:property name="q0_height" value="0.05"/>
     <xacro:property name="q0_limit_lower" value="${-3*pi / 4.0}"/>
@@ -12,5 +12,5 @@
     <xacro:property name="q0_friction" value="0.3"/>
     <xacro:property name="q0_damping" value="0.3"/>
-    <xacro:property name="q1_length" value="0.132"/>
+    <xacro:property name="q1_length" value="0.3"/>
     <xacro:property name="q1_limit_lower" value="${-pi / 4.0}"/>
     <xacro:property name="q1_limit_upper" value="${pi / 2.0}"/>
@@ -19,5 +19,5 @@
     <xacro:property name="q1_friction" value="0.3"/>
     <xacro:property name="q1_damping" value="0.3"/>
-    <xacro:property name="q2_length" value="0.132"/>
+    <xacro:property name="q2_length" value="0.264"/>
     <xacro:property name="q2_limit_lower" value="${-3*pi / 4.0}"/>
     <xacro:property name="q2_limit_upper" value="${3*pi / 4.0}"/>
@@ -27,10 +27,10 @@
     <xacro:property name="q2_damping" value="0.3"/>
     <!-- arm_base_link -->
-    <xacro:cylinder link_name="arm_base_link" m="10.0" o_xyz="0 0 ${q0_height / 2.0}"
-    o_rpy="0 0 0" radius="0.06" length="${q0_height}" material_name="orange"/>
+    <xacro:cylinder link_name="arm_base_link" m="1.0" o_xyz="0 0 ${q0_height / 2.0}"
+    o_rpy="0 0 0" radius="0.16" length="${q0_height}" material_name="orange"/>
     <!-- arm_base_link -->
     <!-- q0 -->
     <xacro:sphere link_name="q0_link" m="0.75" o_xyz="0 0 0" o_rpy="0 0 0"
-    radius="0.05" material_name="orange"/>
+    radius="0.1" material_name="orange"/>
     <joint name="q0" type="revolute">
         <parent link="arm_base_link"/>

File: agv_models/agv_mini_manipulator/agv_mini_manipulator_description/urdf/manipulator/arm_gazebo.xacro (robot description, xacro)
@@ -15,5 +15,6 @@
             name="gz::sim::systems::JointPositionController" >
             <joint_name>q1</joint_name>
-            <p_gain>3.0</p_gain>
+            <p_gain>6.0</p_gain>
+            <d_gain>2.5</d_gain>
         </plugin>
     </gazebo>
@@ -23,5 +24,6 @@
             name="gz::sim::systems::JointPositionController" >
             <joint_name>q2</joint_name>
-            <p_gain>3.0</p_gain>
+            <p_gain>6.0</p_gain>
+            <d_gain>2.5</d_gain>
         </plugin>
     </gazebo>

File: agv_models/agv_mini_manipulator/agv_mini_manipulator_description/urdf/robot.urdf.xacro (robot description, xacro)
@@ -3,7 +3,18 @@
     <xacro:include filename="common_properties.xacro"/>
     <xacro:include filename="common_hardware.xacro"/>
-    <!-- Mobile base -->
-    <!-- <xacro:include filename="$(find agv_mini_manipulator_description)/urdf/mobile_base/mobile_base_robot.urdf.xacro"/> -->
+    <!-- Mobile Base-->
+    <xacro:include filename="$(find agv_mini_manipulator_description)/urdf/mobile_base/mobile_base.xacro"/>
+    <xacro:include filename="$(find agv_mini_manipulator_description)/urdf/mobile_base/mobile_base_gazebo.xacro"/>
+    <!-- Sensors -->
+    <xacro:include filename="$(find agv_mini_manipulator_description)/urdf/sensors/camera.xacro"/>
+    <xacro:include filename="$(find agv_mini_manipulator_description)/urdf/sensors/lidar.xacro"/>
     <!-- Manipulator -->
-    <!-- <xacro:include filename="$(find agv_mini_manipulator_description)/urdf/manipulator/manipulator.urdf.xacro"/> -->
+    <xacro:include filename="$(find agv_mini_manipulator_description)/urdf/manipulator/arm.xacro"/>
+    <xacro:include filename="$(find agv_mini_manipulator_description)/urdf/manipulator/arm_gazebo.xacro"/>
+    <!-- Connection -->
+    <joint name="base_link_to_arm_base_link" type="fixed">
+        <parent link="base_link"/>
+        <child link="arm_base_link"/>
+        <origin xyz="0 0 ${base_height / 2.0}" rpy="0 0 0"/>
+    </joint>
 </robot>
