Commit message: For the agv_mini_manipulator: 1. Simplified manipulator gz bindings. Add functional front gz lidar. Fixed Imu and lidar headings (use gz_frame_id, ignore gz warnings. Depreciated frame_id does not fix headings). Add converted python full robot launch file.

File: agv_models/agv_mini_manipulator/agv_mini_manipulator_description/urdf/manipulator/arm_gazebo.xacro (robot description, xacro)
@@ -2,30 +2,20 @@
 <robot xmlns:xacro="http://www.ros.org/wiki/xacro">
     <!-- Controllers -->
-    <gazebo>
-        <plugin
-            filename="gz-sim-joint-position-controller-system"
-            name="gz::sim::systems::JointPositionController" >
-            <joint_name>q0</joint_name>
-            <p_gain>5.0</p_gain>
-        </plugin>
-    </gazebo>
-    <gazebo>
-        <plugin
-            filename="gz-sim-joint-position-controller-system"
-            name="gz::sim::systems::JointPositionController" >
-            <joint_name>q1</joint_name>
-            <p_gain>6.0</p_gain>
-            <d_gain>2.5</d_gain>
-        </plugin>
-    </gazebo>
-    <gazebo>
-        <plugin
-            filename="gz-sim-joint-position-controller-system"
-            name="gz::sim::systems::JointPositionController" >
-            <joint_name>q2</joint_name>
-            <p_gain>6.0</p_gain>
-            <d_gain>2.5</d_gain>
-        </plugin>
-    </gazebo>
+    <xacro:macro name="joint_position_controller" params="joint_name p_gain i_gain d_gain">
+        <gazebo>
+            <plugin
+                filename="gz-sim-joint-position-controller-system"
+                name="gz::sim::systems::JointPositionController" >
+                <topic>/cmd_pos/${joint_name}</topic>
+                <joint_name>${joint_name}</joint_name>
+                <p_gain>${p_gain}</p_gain>
+                <i_gain>${i_gain}</i_gain>
+                <d_gain>${d_gain}</d_gain>
+            </plugin>
+        </gazebo>
+    </xacro:macro>
+    <xacro:joint_position_controller joint_name="q0" p_gain="5.0" i_gain="0.01" d_gain="0.1"/>
+    <xacro:joint_position_controller joint_name="q1" p_gain="6.0" i_gain="0.01" d_gain="2.5"/>
+    <xacro:joint_position_controller joint_name="q2" p_gain="6.0" i_gain="0.01" d_gain="2.5"/>
     <!-- State publisher -->
     <gazebo>
@@ -33,4 +23,5 @@
             filename="gz-sim-joint-state-publisher-system"
             name="gz::sim::systems::JointStatePublisher" >
+            <topic>joint_states</topic>
             <joint_name>q0</joint_name>
             <joint_name>q1</joint_name>

File: agv_models/agv_mini_manipulator/agv_mini_manipulator_description/urdf/mobile_base/mobile_base.xacro (robot description, xacro)
@@ -27,5 +27,5 @@
         rpy="${pi / 2.0} 0 0"/>
         <axis xyz="0 0 1"/>
-        <effort>20</effort>
+        <limit effort = "20.0" velocity="10.0"/>
     </joint>
     <!-- base_link_right_wheel_joint -->
@@ -38,5 +38,5 @@
         rpy="${pi / 2.0} 0 0"/>
         <axis xyz="0 0 1"/>
-        <effort>20</effort>
+        <limit effort = "20.0" velocity="10.0"/>
     </joint>
     <!-- base_link_left_wheel_joint -->

File: agv_models/agv_mini_manipulator/agv_mini_manipulator_description/urdf/mobile_base/mobile_base_gazebo.xacro (robot description, xacro)
@@ -13,11 +13,17 @@
             filename="gz-sim-diff-drive-system"
             name="gz::sim::systems::DiffDrive" >
+            <!-- Wheel Information -->
             <left_joint>base_link_left_wheel_joint</left_joint>
             <right_joint>base_link_right_wheel_joint</right_joint>
             <wheel_separation>${base_width + wheel_thickness}</wheel_separation>
             <wheel_radius>${wheel_radius}</wheel_radius>
-            <odom_publish_frequency>1</odom_publish_frequency>
+            <!-- Input -->
+            <topic>cmd_vel</topic>
+            <!-- Output -->
             <frame_id>odom</frame_id>
             <child_frame_id>base_footprint</child_frame_id>
+            <odom_topic>odom</odom_topic>
+            <odom_publish_frequency>1</odom_publish_frequency>
+            <tf_topic>tf</tf_topic>
         </plugin>
     </gazebo>
@@ -26,4 +32,5 @@
             filename="gz-sim-joint-state-publisher-system"
             name="gz::sim::systems::JointStatePublisher" >
+            <topic>joint_states</topic>
             <joint_name>base_link_left_wheel_joint</joint_name>
             <joint_name>base_link_right_wheel_joint</joint_name>

File: agv_models/agv_mini_manipulator/agv_mini_manipulator_description/urdf/robot.urdf.xacro (robot description, xacro)
@@ -7,5 +7,5 @@
     <xacro:include filename="$(find agv_mini_manipulator_description)/urdf/mobile_base/mobile_base_gazebo.xacro"/>
     <!-- Sensors -->
-    <xacro:include filename="$(find agv_mini_manipulator_description)/urdf/sensors/camera.xacro"/>
+    <!-- <xacro:include filename="$(find agv_mini_manipulator_description)/urdf/sensors/camera.xacro"/> -->
     <xacro:include filename="$(find agv_mini_manipulator_description)/urdf/sensors/lidar.xacro"/>
     <xacro:include filename="$(find agv_mini_manipulator_description)/urdf/sensors/imu.xacro"/>

File: agv_models/agv_mini_manipulator/agv_mini_manipulator_description/urdf/sensors/imu.xacro (robot description, xacro)
@@ -10,10 +10,10 @@
         <origin xyz="0 0 0" rpy="0 0 0"/>
     </joint>
-    <!-- base_link_imu_joint -->
     <gazebo reference="imu_link">
       <sensor name="imu_sensor" type="imu">
         <always_on>1</always_on>
         <update_rate>50</update_rate>
-        <topic>imu/data</topic>
+        <topic>imu</topic>
+        <gz_frame_id>imu_link</gz_frame_id>
         <imu>
           <enable_orientation>0</enable_orientation>
@@ -97,3 +97,4 @@
         </plugin>
     </gazebo>
+    <!-- base_link_imu_joint -->
 </robot>

File: agv_models/agv_mini_manipulator/agv_mini_manipulator_description/urdf/sensors/lidar.xacro (robot description, xacro)
@@ -14,4 +14,38 @@
     </joint>
     <!-- base_link_lidar_front_joint -->
+    <gazebo reference="front_lidar_link">
+        <sensor name="front_lidar_link" type="gpu_lidar">
+                <topic>laser_scan</topic>
+                <visualize>true</visualize>
+                <update_rate>10</update_rate>
+                <gz_frame_id>front_lidar_link</gz_frame_id>
+                <lidar>
+                    <scan>
+                        <horizontal>
+                        <samples>10</samples>
+                        <resolution>1</resolution>
+                        <min_angle>${-pi / 2.0}</min_angle>
+                        <max_angle>${pi / 2.0}</max_angle>
+                        </horizontal>
+                        <vertical>
+                        <samples>4</samples>
+                        <resolution>1</resolution>
+                        <min_angle>-0.261799</min_angle>
+                        <max_angle>0.261799</max_angle>
+                        </vertical>
+                    </scan>
+                    <range>
+                        <min>0.05</min>
+                        <max>100</max>
+                        <resolution>0.01</resolution>
+                    </range>
+                    <noise>
+                        <type>gaussian</type>
+                        <mean>0</mean>
+                        <stddev>0.01</stddev>
+                    </noise>
+                </lidar>
+            </sensor>
+    </gazebo>
     <!-- base_link_lidar_back_joint -->
     <xacro:cylinder link_name="back_lidar_link" m="0.5" o_xyz="0 0 0" o_rpy="0 0 0"
